File: Led_matrix/Led_matrix.sch (EAGLE design)
At the start: 79 parts, among them J1 DC-005

Commit message: Footprints and schematic modifications
Footprints have been added and the schematic modified.
Parts:
- removed JP10, JP9: (no value), pinhead:PINHD-2X7
- removed JP11, JP12: (no value), pinhead:PINHD-1X14
- removed JP8: (no value), pinhead:PINHD-2X5
- removed R12, R13: (no value), resistor:R-EU_0207/10
- removed SW1: (no value), OPL-Switch:DIP-BUTTON(4P-12.0X12.0X4.2MM)-TS-1103-H4.3MM
- added ASDASDASASD, ASDASDSADSASADSAD: (no value), pinhead:PINHD-1X14
- added C2: 100uf, OPL-Capacitor:DIP-ALUMINUM-100UF-16V(D5-H7MM)
- added D25: 20V-500MA, OPL-Diode:SMD-DIODE-SCHOTTKY-20V-500MA(SOD-123)P
- added GHBGBHG: (no value), pinhead:PINHD-2X5
- added L1: 2.2UH-1.2A, OPL-Inductor:SMD-INDUCTOR-2.2UH-20%-1.2A(0805)
- added SW2: (no value), OPL-Switch:SMD-BUTTON(4P-6.0X6.0X7.5MM)
- added TGFGF: (no value), pinhead:PINHD-2X7
- C1: value (none) -> 100nf; device resistor:C-EU025-050X050 -> OPL-Capacitor:DIP-CERAMIC-DISC-100NF-50V-Y5V(D5.0MM)
- D1, D10, D11, D12, D13, D14, D15, D16, D17, D18, D19, D2, D20, D21, D22, D23, D24, D3, D4, D5, D6, D7, D8, D9: value GREEN-0603 -> (none)
- IC1: value (none) -> ATMEGA88; device ic-package:DIL18 -> custom-ic-package:DIL28-3
- IC2: value (none) -> SN74HC595N; device ic-package:DIL16 -> custom-ic-package:DIL16-SMD
- IC3: value (none) -> ULN2803APG; device ic-package:DIL28 -> custom-ic-package:DIL18-SMD
- JP1: value (none) -> SLAVE_1; device pinhead:PINHD-1X6 -> custom-pinhead:PINHD-2X3-SMD
- JP2: value (none) -> SLAVE_2; device pinhead:PINHD-1X6 -> custom-pinhead:PINHD-2X3-SMD
- JP3: value (none) -> SLAVE_3; device pinhead:PINHD-1X6 -> custom-pinhead:PINHD-2X3-SMD
- JP4: value (none) -> SLAVE_4; device pinhead:PINHD-1X6 -> custom-pinhead:PINHD-2X3-SMD
- JP5: value (none) -> MASTER; device pinhead:PINHD-1X6 -> custom-pinhead:PINHD-2X3-SMD
- JP6: value (none) -> ISP; device pinhead:PINHD-2X3 -> custom-pinhead:PINHD-2X3-SHROUDED
- R15, R16, R17, R18, R19, R20, R21, R22, R23, R24, R25, R26, R27, R28, R29, R30, R31, R32, R33, R34, R35, R36, R37: value 100R -> (none)
- renumbered JP7 to ERQWEWEW
Connections:
- new net GND: C1.2, SW2.B0
- new net N$1: C1.1, IC1.1, R11.2, SW2.A0
- new net VDD: R11.1
Other:
- note added: "Debug av I/O:s av samtliga Atmega88:or"
- note added: "Free-wheel-diode for the low pass filter"
- note added: "GameController"
- note added: "ISP"
- note added: "LED MATRIX 8x6 segment signals"
- note added: "MASTER: I2C, GND, VDD, DUMMIES"
- note added: "Powersource"
- note added: "SLAVES: I2C, GND, VDD, DUMMIES"
- note removed: "DC led status"
- note removed: "STIFTLISTER"
- moved on the sheet: D1, D10, D11, D12, D13, D14, D15, D16, D17, D18, D19, D2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
